File: kicad/PSN_TRX.kicad_sch (KiCad schematic)
At the start: 150 parts, among them IC1 LP2950L-5.0V, IC2 NJM2904, J1 PWR_IN, J2 SP-OUT, J3 RF-IN, J4 MIC-IN, J5 I2C_OUT, J6 Volume, K1 G5V-2, Q1 3SK59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

Commit message: feat: assign GF063P footprint to VR3-VR7
Parts:
- VR3, VR4, VR5, VR6, VR7: footprint Potentiometer_THT:Potentiometer_Alps_RK09K_Single_Vertical -> PSN_TRX:Potentiometer_TOCOS_GF063P_Vertical
Changed lines of the file:
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@@
 			)
 		)
-		(property "Footprint" "Potentiometer_THT:Potentiometer_Alps_RK09K_Single_Vertical"
+		(property "Footprint" "PSN_TRX:Potentiometer_TOCOS_GF063P_Vertical"
 			(at 612.14 358.14 0)
 			(hide yes)
@@
 			)
 		)
-		(property "Footprint" "Potentiometer_THT:Potentiometer_Alps_RK09K_Single_Vertical"
+		(property "Footprint" "PSN_TRX:Potentiometer_TOCOS_GF063P_Vertical"
 			(at 600.71 438.15 0)
 			(hide yes)
@@
 			)
 		)
-		(property "Footprint" "Potentiometer_THT:Potentiometer_Alps_RK09K_Single_Vertical"
+		(property "Footprint" "PSN_TRX:Potentiometer_TOCOS_GF063P_Vertical"
 			(at 421.64 358.14 0)
 			(hide yes)
@@
 			)
 		)
-		(property "Footprint" "Potentiometer_THT:Potentiometer_Alps_RK09K_Single_Vertical"
+		(property "Footprint" "PSN_TRX:Potentiometer_TOCOS_GF063P_Vertical"
 			(at 421.64 328.93 0)
 			(hide yes)
@@
 			)
 		)
-		(property "Footprint" "Potentiometer_THT:Potentiometer_Alps_RK09K_Single_Vertical"
+		(property "Footprint" "PSN_TRX:Potentiometer_TOCOS_GF063P_Vertical"
 			(at 609.6 328.93 0)
 			(hide yes)
