File: kicad/PSN_TRX.kicad_sch (KiCad schematic)
At the start: 163 parts, among them IC1 LP2950L-5.0V, IC2 NJM2904, J1 RF_IN, J2 SP-OUT, J3 PWR_IN, J4 Volume, J5 Volume, J6 Conn_01x04, J7 I2C_OUT, J8 MIC-IN, K1 G5V-2, Q1 2SC2120, Q10 2SK439, Q11 2SC1815, Q12 2SC1815, Q13 2SC1815, Q14 2SC1815, Q2 2SC1815, Q3 BF998, Q4 2SC1923, Q5 2SC1815, Q6 2SA950, Q7 2SK439, Q8 RD06HVF1, Q9 2SC1815, SW1 SW, SW2 SW, T1 ST-71, U1 LP2950-3.3_TO92, U2 Si5351_DIP8

Commit message: update: KiCadで手動変更した回路図・PCB・プロジェクトファイルを反映
Q3 BF998換装・バイアス回路変更等のKiCad GUI編集内容をコミット。

Co-Authored-By: Claude Sonnet 4.6 <noreply@anthropic.com>
Parts:
- removed Q3: BF998, Package_TO_SOT_SMD:SOT-143, symbol Transistor_FET:3SK263
- added Q3: BF998, PSN_TRX:BF998_SOT143, symbol PSN_TRX:BF998
Connections:
- net at C12.1, L2.1 (SA): now also Q3.1 (G1)
- net at C13.1, J5.2 (Pin_2): now also Q3.3 (G2)
- net at C15.1, R13.1: now also Q3.2 (S)
- net at C6.1, L1.4 (AA): now also Q3.4 (D)
Changed lines of the file:
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@@
+	)
+	(symbol
+		(lib_id "PSN_TRX:BF998")
+		(at 213.36 124.46 0)
+		(unit 1)
+		(body_style 1)
+		(exclude_from_sim no)
+		(in_bom yes)
+		(on_board yes)
+		(in_pos_files yes)
+		(dnp no)
+		(fields_autoplaced yes)
+		(property "Reference" "Q3"
+			(at 219.71 123.1899 0)
+			(show_name no)
+			(do_not_autoplace no)
+			(effects
+				(font
+					(size 1.27 1.27)
+				)
+				(justify left)
+			)
+		)
+		(property "Value" "BF998"
+			(at 219.71 125.7299 0)
+			(show_name no)
+			(do_not_autoplace no)
+			(effects
+				(font
+					(size 1.27 1.27)
+				)
+				(justify left)
+			)
+		)
+		(property "Footprint" "PSN_TRX:BF998_SOT143"
+			(at 218.44 126.365 0)
+			(hide yes)
+			(show_name no)
+			(do_not_autoplace no)
+			(effects
+				(font
+					(size 1.27 1.27)
+				)
+				(justify left)
+			)
+		)
+		(property "Datasheet" "https://www.nxp.com/docs/en/data-sheet/BF998.pdf"
+			(at 218.44 128.27 0)
+			(hide yes)
+			(show_name no)
+			(do_not_autoplace no)
+			(effects
+				(font
+					(size 1.27 1.27)
+				)
+				(justify left)
+			)
+		)
+		(property "Description" "N-Ch Dual Gate Depletion MOSFET, 12V Vds, 30mA, SOT-143"
+			(at 213.36 124.46 0)
+			(hide yes)
+			(show_name no)
+			(do_not_autoplace no)
+			(effects
+				(font
+					(size 1.27 1.27)
+				)
+			)
+		)
+		(pin "1"
+		)
+		(pin "2"
+		)
+		(pin "4"
+		)
+		(pin "3"
+		)
+		(instances
+			(project "PSN_TRX"
+				(path "/50835569-93ad-4c8c-aafc-424a6a3761ef"
+					(reference "Q3")
+					(unit 1)
+				)
+			)
+		)
 	)
 	(symbol
@@
 					(unit 1)
 				)
-			)
-		)
-	)
-	(symbol
-		(lib_id "Transistor_FET:3SK263")
-		(at 213.36 124.46 0)
-		(unit 1)
-		(body_style 1)
-		(exclude_from_sim no)
-		(in_bom yes)
-		(on_board yes)
-		(in_pos_files yes)
-		(dnp no)
-		(property "Reference" "Q3"
-			(at 211.836 113.792 0)
-			(show_name no)
-			(do_not_autoplace no)
-			(effects
-				(font
-					(size 1.27 1.27)
-				)
-			)
-		)
-		(property "Value" "BF998"
-			(at 217.932 113.538 0)
-			(show_name no)
-			(do_not_autoplace no)
-			(effects
-				(font
-					(size 1.27 1.27)
-				)
-			)
-		)
-		(property "Footprint" "Package_TO_SOT_SMD:SOT-143"
-			(at 213.36 124.46 0)
-			(hide yes)
-			(show_name no)
-			(do_not_autoplace no)
-			(effects
-				(font
-					(size 1.27 1.27)
-				)
-			)
-		)
-		(property "Datasheet" ""
-			(at 213.36 124.46 0)
-			(hide yes)
-			(show_name no)
-			(do_not_autoplace no)
-			(effects
-				(font
-					(size 1.27 1.27)
-				)
-			)
-		)
-		(property "Description" ""
-			(at 213.36 124.46 0)
-			(show_name no)
-			(do_not_autoplace no)
-			(effects
-				(font
-					(size 1.27 1.27)
-				)
-			)
-		)
-		(property "ki_description" "高周波増幅"
-			(at 213.36 124.46 0)
-			(hide yes)
-			(show_name no)
-			(do_not_autoplace no)
-			(effects
-				(font
-					(size 1.27 1.27)
-				)
-			)
-		)
-		(pin "1"
-		)
-		(pin "2"
-		)
-		(pin "4"
-		)
-		(pin "3"
-		)
-		(instances
-			(project "PSN_TRX"
-				(path "/50835569-93ad-4c8c-aafc-424a6a3761ef"
-					(reference "Q3")
-					(unit 1)
-				)

Commit message: Rename project from PSN_TRX_Nano_R4 to PSN_TRX_XIAO_SAMD21
- Update README.md title
- Update KiCad project files

Co-Authored-By: Claude Haiku 4.5 <noreply@anthropic.com>
Connections:
- net +9V: now also L1.3 (SB); no longer L1.5 (AB)
- net GND: now also L1.5 (AB); no longer L1.3 (SB)
- net at L1.1 (SA): now also C6.1, Q3.4 (D); no longer C7.1
- new net: C7.1, L1.4 (AA)
Changed lines of the file:
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@@
 	)
 	(no_connect
-		(at 265.43 123.19)
+		(at 245.11 123.19)
 	)
 	(no_connect
@@
 		(lib_id "PSN_TRX:L_7T50_CT")
 		(at 255.27 123.19 0)
+		(mirror y)
 		(unit 1)
 		(body_style 1)
@@
 		(dnp no)
 		(property "Reference" "L1"
-			(at 253.492 112.268 0)
+			(at 257.048 112.268 0)
 			(show_name no)
 			(do_not_autoplace no)
@@
 		)
 		(property "Value" "7T50"
-			(at 258.318 112.268 0)
+			(at 252.222 112.268 0)
 			(show_name no)
 			(do_not_autoplace no)

Commit message: Update component footprints and settings
- LED2: set on_board to 'no'
- R21, R22: change footprint from P10.16mm_Horizontal to P5.08mm_Vertical

Co-Authored-By: Claude Haiku 4.5 <noreply@anthropic.com>
Parts:
- removed C26: 1000pF, Capacitor_THT:C_Disc_D5.0mm_W2.5mm_P5.00mm, symbol Device:C
- added J9: TX-ON-LED, Connector_PinHeader_2.54mm:PinHeader_1x02_P2.54mm_Vertical, symbol Connector_Generic:Conn_01x02
- R21, R22: footprint Resistor_THT:R_Axial_DIN0207_L6.3mm_D2.5mm_P10.16mm_Horizontal -> Resistor_THT:R_Axial_DIN0207_L6.3mm_D2.5mm_P5.08mm_Vertical
Connections:
- net at C27.1, C30.2, C32.1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: no longer LED2.2 (A)
- new net: J9.1 (Pin_1), Q11.2 (C)
- new net: J9.2 (Pin_2), R25.1
- now unconnected: LED2.1 (K)
Other:
- moved on the sheet: C50, C51, C52, C53, C54, C55, C56, C57, C58, C59, C60, IC2A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
