File: kicad/PSN_TRX.kicad_pcb (KiCad board)
At the start: 4 copper layers, 220 x 150 mm, 156 parts, among them IC1 LP2950L-5.0V, IC2 NJM2904, J1 RF_IN, J2 SP-OUT, J3 PWR_IN, J4 Volume, J5 Volume, J6 Conn_01x04, J7 I2C_OUT, J8 MIC-IN, J9 TX-ON-LED, K1 G5V-2, Q1 2SC2120, Q10 2SK439, Q11 2SC1815, Q12 2SC1815, Q13 2SC1815, Q14 2SC1815, Q2 2SC1815, Q3 BF998, Q4 2SC1923, Q5 2SC1815, Q6 2SA950, Q7 2SK439, Q8 RD06HVF1, Q9 2SC1815, T1 ST-71, U1 LP2950-3.3_TO92, U2 Si5351_DIP8

Commit message: update: 回路図・PCBを更新
- I2C_OUTコネクタをI2C_OUT-LCDにリネーム
- EncoderコネクタのValueをConn_01x04からEncoderに変更
- PCBレイアウト更新

Co-Authored-By: Claude Sonnet 4.6 <noreply@anthropic.com>
Parts:
- added J10: TJC4832T135, Connector_PinHeader_2.54mm:PinHeader_1x04_P2.54mm_Vertical, F.Cu at (206.5, 69.7)
- J6: value Conn_01x04 -> Encoder
- J7: value I2C_OUT -> I2C_OUT-LCD
- Studio XIAO ESP32C3: renamed from A1
- moved J6 206.4 mm to (206.5, 52.5)
- moved J2 51.7 mm to (206.5, 38.9)
- moved U2 36.1 mm to (172.3, 67.3)
- moved J7 30.5 mm to (206.5, 89.0)
- moved Studio XIAO ESP32C3 28.9 mm to (191.3, 69.1)
- moved IC2 17.5 mm to (164.9, 100.4)
- moved C11 15.0 mm to (172.5, 40.0)
Connections:
- Studio XIAO ESP32C3 pad 14: unconnected-(A1-D7/RX-Pad14) -> Net-(J10-Pin_3)
- Studio XIAO ESP32C3 pad 7: unconnected-(A1-D6/TX-Pad7) -> Net-(J10-Pin_2)
