File: transceiver/PSN_TRX.kicad_sch (KiCad schematic)
At the start: 159 parts, among them IC1 LP2950L-5.0V, IC2 NJM2904, J1 PWR_IN, K1 G5V-2, Q1 3SK59, Q10 2SK439, Q11 2SC1815, Q12 2SC1815, Q13 2SC1815, Q14 2SK439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

Commit message: feat: assign GF063P footprint to VR3-VR5
Parts:
- VR3, VR4, VR5: footprint Potentiometer_THT:Potentiometer_Alps_RK09K_Single_Vertical -> PSN_TRX:Potentiometer_TOCOS_GF063P_Vertical
Changed lines of the file:
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@@
 			)
 		)
-		(property "Footprint" "Potentiometer_THT:Potentiometer_Alps_RK09K_Single_Vertical"
+		(property "Footprint" "PSN_TRX:Potentiometer_TOCOS_GF063P_Vertical"
 			(at 565.15 416.56 0)
 			(hide yes)
@@
 			)
 		)
-		(property "Footprint" "Potentiometer_THT:Potentiometer_Alps_RK09K_Single_Vertical"
+		(property "Footprint" "PSN_TRX:Potentiometer_TOCOS_GF063P_Vertical"
 			(at 382.27 336.55 0)
 			(hide yes)
@@
 			)
 		)
-		(property "Footprint" "Potentiometer_THT:Potentiometer_Alps_RK09K_Single_Vertical"
+		(property "Footprint" "PSN_TRX:Potentiometer_TOCOS_GF063P_Vertical"
 			(at 382.27 307.34 0)
 			(hide yes)
