File: transceiver/PSN_TRX.kicad_sch (KiCad schematic)
At the start: 159 parts, among them IC1 LP2950L-5.0V, IC2 NJM2904, J1 PWR_IN, K1 G5V-2, Q1 3SK59, Q10 2SK439, Q11 2SC1815, Q12 2SC1815, Q13 2SC1815, Q14 2SK439, Q15 2SC1815, Q17 2SC1815, Q2 2SC1923, Q3 2SC1815, Q4 2SC1815, Q5 2SC2120, Q6 2SA950, Q7 2SC1923, Q8 2SC1923, Q9 2SK439, SW1 SW, T1 ST-71, X1 50.5MHz/3

Commit message: fix: VR1/VR2 を DNP・NO board に設定（in_bom/on_board/in_pos_files=no, dnp=yes）
Co-Authored-By: Claude Sonnet 4.6 <noreply@anthropic.com>
Parts:
- VR1, VR2: now not fitted; now left out of the parts list
Changed lines of the file:
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@@
 		(body_style 1)
 		(exclude_from_sim no)
-		(in_bom yes)
-		(on_board yes)
-		(in_pos_files yes)
-		(dnp no)
+		(in_bom no)
+		(on_board no)
+		(in_pos_files no)
+		(dnp yes)
 		(property "Reference" "VR2"
 			(at 517.398 77.978 0)
@@
 		(body_style 1)
 		(exclude_from_sim no)
-		(in_bom yes)
-		(on_board yes)
-		(in_pos_files yes)
-		(dnp no)
+		(in_bom no)
+		(on_board no)
+		(in_pos_files no)
+		(dnp yes)
 		(fields_autoplaced yes)
 		(property "Reference" "VR1"
